File: thumb-keyboard/thumb-keyboard.kicad_pcb (KiCad board)
At the start: 2 copper layers, 144 x 60 mm, 201 parts, among them J1 Conn_01x02_Socket, U1 nice_nano

Commit message: finishing migrating to thummingboard repo
Parts:
- G***: footprint thummingbird:thummingbird -> thummingbirdlogo:thummingbird
Changed lines of the file:
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@@
 		)
 	)
-	(footprint "thummingbird:thummingbird"
+	(footprint "thummingbirdlogo:thummingbird"
 		(layer "B.Cu")
 		(at 103.5 85.5 180)
 		(property "Reference" "G***"
 			(at 0 0 0)
-			(layer "F.SilkS")
+			(layer "B.SilkS")
 			(hide yes)
 			(effects
