File: thumb-keyboard/thumb-keyboard.kicad_sch (KiCad schematic)
At the start: 192 parts, among them J1 Conn_01x02_Socket, U1 nice_nano

Commit message: small maintenence
Parts:
- S1: value ESC -> PTS526 SK15 SMTR2 LFS
Changed lines of the file:
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@@
 			)
 		)
-		(property "Value" "ESC"
+		(property "Value" "PTS526 SK15 SMTR2 LFS"
 			(at 129.54 38.1 0)
 			(effects
